Commit message: Đã cập nhật URDF cho robot

File: description/bena.urdf.xacro (robot description, xacro)
@@ -2,3 +2,5 @@
 <robot xmlns:xacro="http://www.ros.org/wiki/xacro"  name="robot">
     <xacro:include filename = "bena_core.xacro"/>
+    <xacro:include filename = "gazebo_control.xacro"/>
+    <xacro:include filename = "lidar.xacro"/>
 </robot>

File: description/bena_core.xacro (robot description, xacro)
@@ -17,4 +17,12 @@
     <link name="base_link">
     </link>
+    <!-- BASE_FOOTPRINT LINK -->
+     <joint name = "base_footprint_joint" type="fixed">
+        <parent link="base_link"/>
+        <child link="base_footprint"/>
+        <origin xyz="0 0 0 " rpy =" 0 0 0"/><!--hinh chieu len mat phang day, tham chieu vi tri cua robot-->
+     </joint>
+     <link name = "base_footprint">
+     </link>
     <!-- KHUNG LINK-->
     <joint name="khung" type="fixed">
@@ -42,4 +50,7 @@
         </xacro:quan_tinh_hop>
     </link>
+    <gazebo reference="khung">
+        <material>Gazebo/Yellow</material>
+    </gazebo>
     <!-- banh trai LINK-->
      <joint name = "khop_banh_trai" type = "continuous">
@@ -66,4 +77,7 @@
          </xacro:quan_tinh_tru>
      </link>
+     <gazebo reference="banh_trai">
+        <material>Gazebo/Blue</material>
+    </gazebo>
      <!-- banh phai LINK-->
      <joint name = "khop_banh_phai" type = "continuous">
@@ -90,6 +104,9 @@
          </xacro:quan_tinh_tru>
      </link>
+     <gazebo reference="banh_phai">
+        <material>Gazebo/Blue</material>
+    </gazebo>
      <!-- BANH LAN-->
-      <joint name ="khop banh lan" type = "fixed" >
+      <joint name ="khop_banh_lan" type = "fixed" >
         <parent link = "base_link"/>
         <child link = "banh_lan"/>
@@ -113,3 +130,8 @@
          </xacro:quan_tinh_cau>
       </link>
+      <gazebo reference="banh_lan">
+        <material>Gazebo/Red</material>
+        <mu1  value = "0.001"/>
+        <mu2 value = "0.001"/>
+    </gazebo>
 </robot>
