Commit message: Thông điệp commit

File: description/bena_core.xacro (robot description, xacro)
@@ -111,5 +111,5 @@
         <parent link = "base_link"/>
         <child link = "banh_lan"/>
-        <origin xyz = "0.14 0 0"/>
+        <origin xyz = "0.18 0 0"/>
       </joint>
       <link name = "banh_lan">

File: description/lidar.xacro (robot description, xacro)
@@ -38,5 +38,5 @@
                 <range>
                     <min>0.3</min>
-                    <max>12</max>
+                    <max>7</max>
                 </range>
             </ray>
